Commit message: manual adapt fr3

File: franka_description/robots/fr3_arm.ros2_control.xacro (robot description, xacro)
@@ -1,5 +1,5 @@
 <?xml version="1.0"?>
 <robot xmlns:xacro="http://www.ros.org/wiki/xacro">
-  <xacro:macro name="panda_arm_ros2_control" params="ns robot_ip use_fake_hardware:=^|false fake_sensor_commands:=^|false">
+  <xacro:macro name="fr3_arm_ros2_control" params="ns robot_ip use_fake_hardware:=^|false fake_sensor_commands:=^|false">
     <ros2_control name="FrankaHardwareInterface" type="system">
       <hardware>

File: franka_description/robots/fr3_arm.urdf.xacro (robot description, xacro)
@@ -1,16 +1,16 @@
 <?xml version='1.0' encoding='utf-8'?>
-<robot xmlns:xacro="http://www.ros.org/wiki/xacro" name="panda">
-  <xacro:arg name="arm_id" default="panda"/> <!-- Name of this panda -->
+<robot xmlns:xacro="http://www.ros.org/wiki/xacro" name="fr3">
+  <xacro:arg name="arm_id" default="fr3"/> <!-- Name of this fr3 -->
   <xacro:arg name="hand" default="false"/> <!-- Should a franka_gripper be mounted at the flange?" -->
   <xacro:arg name="robot_ip" default=""/> <!-- IP address or hostname of the robot" -->
   <xacro:arg name="use_fake_hardware" default="false"/>
   <xacro:arg name="fake_sensor_commands" default="false"/>
-  <xacro:include filename="$(find franka_description)/robots/panda_arm.xacro"/>
-  <xacro:panda_arm arm_id="$(arg arm_id)" safety_distance="0.03"/>
+  <xacro:include filename="$(find franka_description)/robots/fr3_arm.xacro"/>
+  <xacro:fr3_arm arm_id="$(arg arm_id)" safety_distance="0.03"/>
   <xacro:if value="$(arg hand)">
     <xacro:include filename="$(find franka_description)/robots/hand.xacro"/>
     <xacro:hand ns="$(arg arm_id)" rpy="0 0 ${-pi/4}" connected_to="$(arg arm_id)_link8" safety_distance="0.03"/>
   </xacro:if>
-  <xacro:include filename="$(find franka_description)/robots/panda_arm.ros2_control.xacro"/>
-  <xacro:panda_arm_ros2_control ns="$(arg arm_id)" robot_ip="$(arg robot_ip)" use_fake_hardware="$(arg use_fake_hardware)" fake_sensor_commands="$(arg fake_sensor_commands)"/>
+  <xacro:include filename="$(find franka_description)/robots/fr3_arm.ros2_control.xacro"/>
+  <xacro:fr3_arm_ros2_control ns="$(arg arm_id)" robot_ip="$(arg robot_ip)" use_fake_hardware="$(arg use_fake_hardware)" fake_sensor_commands="$(arg fake_sensor_commands)"/>
 </robot>

File: franka_description/robots/fr3_arm.xacro (robot description, xacro)
@@ -1,7 +1,7 @@
 <?xml version='1.0' encoding='utf-8'?>
-<robot xmlns:xacro="http://www.ros.org/wiki/xacro" name="panda">
+<robot xmlns:xacro="http://www.ros.org/wiki/xacro" name="fr3">
   <!-- safety_distance: Minimum safety distance in [m] by which the collision volumes are expanded and which is enforced during robot motions -->
-  <!-- arm_id: Namespace of the panda arm. Serves to differentiate between arms in case of multiple instances. -->
-  <xacro:macro name="panda_arm" params="arm_id:='panda' description_pkg:='franka_description' connected_to:='' xyz:='0 0 0' rpy:='0 0 0' safety_distance:=0">
+  <!-- arm_id: Namespace of the fr3 arm. Serves to differentiate between arms in case of multiple instances. -->
+  <xacro:macro name="fr3_arm" params="arm_id:='fr3' description_pkg:='franka_description' connected_to:='' xyz:='0 0 0' rpy:='0 0 0' safety_distance:=0">
     <xacro:unless value="${not connected_to}">
       <joint name="${arm_id}_joint_${connected_to}" type="fixed">

File: franka_description/robots/hand.urdf.xacro (robot description, xacro)
@@ -2,4 +2,4 @@
 <robot xmlns:xacro="http://www.ros.org/wiki/xacro" name="hand">
   <xacro:include filename="hand.xacro"/>
-  <xacro:hand ns="panda" safety_distance="0.03"/>
+  <xacro:hand ns="fr3" safety_distance="0.03"/>
 </robot>

File: franka_moveit_config/srdf/panda_arm.srdf.xacro (robot description, xacro)
@@ -1,14 +1,14 @@
 <?xml version='1.0' encoding='utf-8'?>
-<robot xmlns:xacro="http://www.ros.org/wiki/xacro" name="panda">
-  <xacro:arg name="arm_id" default="panda"/> <!-- Name of this panda -->
+<robot xmlns:xacro="http://www.ros.org/wiki/xacro" name="fr3">
+  <xacro:arg name="arm_id" default="fr3"/> <!-- Name of this fr3 -->
   <xacro:arg name="hand" default="true"/> <!-- Should a franka_gripper be mounted at the flange? (Currently does not work without it) -->
   <xacro:property name="arm_id" value="$(arg arm_id)"/>
-  <xacro:include filename="$(find franka_moveit_config)/srdf/panda_arm.xacro"/>
-  <xacro:panda_arm arm_id="${arm_id}"/>
+  <xacro:include filename="$(find franka_moveit_config)/srdf/fr3_arm.xacro"/>
+  <xacro:fr3_arm arm_id="${arm_id}"/>
   <xacro:if value="$(arg hand)">
     <xacro:include filename="$(find franka_moveit_config)/srdf/hand.xacro"/>
     <xacro:hand arm_id="${arm_id}"/>
-    <xacro:include filename="$(find franka_moveit_config)/srdf/panda_arm_hand.xacro"/>
-    <xacro:panda_arm_hand arm_id="${arm_id}"/>
+    <xacro:include filename="$(find franka_moveit_config)/srdf/fr3_arm_hand.xacro"/>
+    <xacro:fr3_arm_hand arm_id="${arm_id}"/>
   </xacro:if>
 </robot>

File: franka_moveit_config/srdf/panda_arm.xacro (robot description, xacro)
@@ -1,5 +1,5 @@
 <?xml version="1.0" ?>
-<robot xmlns:xacro="http://www.ros.org/wiki/xacro" name="panda">
-  <xacro:macro name="panda_arm" params="arm_id:='panda' ">
+<robot xmlns:xacro="http://www.ros.org/wiki/xacro" name="fr3">
+  <xacro:macro name="fr3_arm" params="arm_id:='fr3' ">
     <xacro:include filename="$(find franka_moveit_config)/srdf/group_definition.xacro"/>
     <xacro:group_definition arm_id="${arm_id}" group_name="${arm_id}_manipulator" tip_link="${arm_id}_hand_tcp"/>
